File: circuits/In3Peltier/in3peltier.brd (EAGLE design)
At the start: 45.4 x 39.3 mm, 10 parts

Commit message: Electronics v2
Parts:
- removed R1, R2: 1M, 01_FAB_Hello:1206
- removed U$3, U$4: (no value), 01_FAB_Hello:1206
- moved SL2 7.57 mm to (12.9, 13.3)
- moved C1 4.34 mm to (13.0, 24.0)
Connections:
- removed net N$3: R1.1, U$3.1
- removed net N$4: R2.1, U$4.1
- net BLACK: no longer R2.2
- net GNDH: no longer U$3.2, U$4.2
- net RED: no longer R1.2
Routing:
- net GNDH: track 67.8 -> 39.2 mm
- net BLACK: track 19.5 -> 16.1 mm
- net 12H: track 80.6 -> 84.0 mm
- net N$4: track 3.23 -> 0.00 mm
- net N$3: track 2.89 -> 0.00 mm
Changed lines of the file:
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@@
 <attribute name="OC_FARNELL" value="unknown" x="12.4206" y="2.413" size="1.778" layer="27" display="off"/>
 </element>
-<element name="C1" library="01_SparkFun" package="CPOL-RADIAL-10UF-25V" value="" x="12.954" y="28.3464" rot="R180"/>
-<element name="U$3" library="01_FAB_Hello" package="1206" value="" x="14.0462" y="10.9982" rot="R270"/>
-<element name="U$4" library="01_FAB_Hello" package="1206" value="" x="11.5824" y="10.9982" rot="R270"/>
-<element name="R1" library="01_FAB_Hello" package="1206" value="1M" x="16.764" y="13.9954" rot="R90"/>
-<element name="R2" library="01_FAB_Hello" package="1206" value="1M" x="8.6614" y="13.7414" rot="R90"/>
+<element name="C1" library="01_SparkFun" package="CPOL-RADIAL-10UF-25V" value="" x="12.954" y="24.003" rot="R180"/>
 <element name="SL4" library="con-amp-quick" package="03P" value="" x="12.6492" y="35.6616" rot="R180">
 <attribute name="OC_NEWARK" value="unknown" x="12.6492" y="35.6616" size="1.778" layer="27" rot="R180" display="off"/>
@@
 <element name="U$1" library="0001_alejandro" package="RELAY-V23092" value="RELAY-V23092THROUGH_HOLE" x="20.5994" y="32.9438" rot="R270"/>
 <element name="U$2" library="0001_alejandro" package="RELAY-V23092" value="RELAY-V23092THROUGH_HOLE" x="1.5494" y="33.0454" rot="R270"/>
-<element name="SL2" library="con-amp-quick" package="03P" value="" x="12.9032" y="20.9042">
-<attribute name="OC_NEWARK" value="unknown" x="12.9032" y="20.9042" size="1.778" layer="27" display="off"/>
-<attribute name="MPN" value="" x="12.9032" y="20.9042" size="1.778" layer="27" display="off"/>
-<attribute name="MF" value="" x="12.9032" y="20.9042" size="1.778" layer="27" display="off"/>
-<attribute name="OC_FARNELL" value="unknown" x="12.9032" y="20.9042" size="1.778" layer="27" display="off"/>
+<element name="SL2" library="con-amp-quick" package="03P" value="" x="12.9032" y="13.335">
+<attribute name="OC_NEWARK" value="unknown" x="12.9032" y="13.335" size="1.778" layer="27" display="off"/>
+<attribute name="MPN" value="" x="12.9032" y="13.335" size="1.778" layer="27" display="off"/>
+<attribute name="MF" value="" x="12.9032" y="13.335" size="1.778" layer="27" display="off"/>
+<attribute name="OC_FARNELL" value="unknown" x="12.9032" y="13.335" size="1.778" layer="27" display="off"/>
 </element>
 </elements>
@@
 <contactref element="U$1" pad="2"/>
 <contactref element="U$2" pad="2"/>
-<wire x1="10.1092" y1="35.6616" x2="10.1092" y2="28.3464" width="1.27" layer="1"/>
-<wire x1="10.1092" y1="28.3464" x2="11.684" y2="28.3464" width="1.27" layer="1"/>
 <wire x1="21.5994" y1="20.9438" x2="25.7302" y2="20.9438" width="1.27" layer="1"/>
 <wire x1="25.7302" y1="20.9438" x2="25.7302" y2="39.0398" width="1.27" layer="1"/>
 <wire x1="25.7302" y1="39.0398" x2="10.1092" y2="39.0398" width="1.27" layer="1"/>
-<wire x1="10.1092" y1="38.862" x2="10.1092" y2="35.6616" width="1.27" layer="1"/>
+<wire x1="10.1092" y1="39.0398" x2="10.1092" y2="35.6616" width="1.27" layer="1"/>
 <wire x1="2.5494" y1="21.0454" x2="0.0762" y2="21.0454" width="1.27" layer="1"/>
 <wire x1="0.0762" y1="21.0454" x2="0.0762" y2="39.0398" width="1.27" layer="1"/>
 <wire x1="0.0762" y1="39.0398" x2="10.1092" y2="39.0398" width="1.27" layer="1"/>
-<wire x1="10.1092" y1="39.0398" x2="10.1092" y2="38.862" width="1.27" layer="1"/>
+<wire x1="10.1092" y1="35.6616" x2="10.1092" y2="25.5778" width="1.016" layer="1"/>
+<wire x1="10.1092" y1="25.5778" x2="11.684" y2="24.003" width="1.016" layer="1"/>
 </signal>
 <signal name="GNDH">
 <contactref element="C1" pad="2"/>
-<contactref element="U$3" pad="2"/>
-<contactref element="U$4" pad="2"/>
-<wire x1="11.5824" y1="9.5762" x2="14.0462" y2="9.5762" width="1.4224" layer="1"/>
-<wire x1="14.1986" y1="9.5762" x2="14.0462" y2="9.5762" width="1.4224" layer="1"/>
 <contactref element="SL4" pad="1"/>
 <contactref element="U$1" pad="1"/>
 <contactref element="U$2" pad="1"/>
 <wire x1="15.1892" y1="35.6616" x2="15.1892" y2="30.9372" width="1.27" layer="1"/>
-<wire x1="15.1892" y1="30.9372" x2="15.1892" y2="28.3464" width="1.27" layer="1"/>
-<wire x1="15.1892" y1="28.3464" x2="14.224" y2="28.3464" width="1.27" layer="1"/>
 <wire x1="21.5994" y1="30.9438" x2="20.1008" y2="30.9372" width="1.27" layer="1"/>
 <wire x1="20.1008" y1="30.9372" x2="15.1892" y2="30.9372" width="1.27" layer="1"/>
-<wire x1="2.5494" y1="31.0454" x2="2.5494" y2="30.9372" width="1.27" layer="1"/>
-<wire x1="2.5494" y1="30.9372" x2="6.985" y2="30.9372" width="1.27" layer="1"/>
-<wire x1="6.985" y1="30.9372" x2="6.985" y2="25.8318" width="1.27" layer="1"/>
-<wire x1="6.985" y1="25.8318" x2="14.351" y2="25.8318" width="1.27" layer="1"/>
-<wire x1="14.351" y1="25.8318" x2="14.351" y2="28.3464" width="1.27" layer="1"/>
-<wire x1="14.351" y1="28.3464" x2="14.224" y2="28.3464" width="1.27" layer="1"/>
-<wire x1="14.1986" y1="9.5762" x2="17.6026" y2="9.5762" width="1.27" layer="1"/>
-<wire x1="17.6026" y1="9.5762" x2="19.8374" y2="11.811" width="1.27" layer="1"/>
-<wire x1="19.8374" y1="11.811" x2="19.8374" y2="18.034" width="1.27" layer="1"/>
-<wire x1="19.8374" y1="18.034" x2="18.6436" y2="19.2278" width="1.27" layer="1"/>
-<wire x1="18.6436" y1="19.2278" x2="18.6436" y2="21.8694" width="1.27" layer="1"/>
-<wire x1="18.6436" y1="21.8694" x2="20.3962" y2="23.622" width="1.27" layer="1"/>
-<wire x1="20.3962" y1="23.622" x2="22.9362" y2="23.622" width="1.27" layer="1"/>
-<wire x1="22.9362" y1="23.622" x2="23.9014" y2="24.5872" width="1.27" layer="1"/>
-<wire x1="23.9014" y1="24.5872" x2="23.9014" y2="28.6418" width="1.27" layer="1"/>
-<wire x1="23.9014" y1="28.6418" x2="21.5994" y2="30.9438" width="1.27" layer="1"/>
+<wire x1="15.1892" y1="30.9372" x2="15.1892" y2="24.9682" width="1.016" layer="1"/>
+<wire x1="15.1892" y1="24.9682" x2="14.224" y2="24.003" width="1.016" layer="1"/>
+<wire x1="2.5494" y1="31.0454" x2="2.5494" y2="29.4292" width="1.016" layer="1"/>
+<wire x1="2.5494" y1="29.4292" x2="11.6586" y2="20.32" width="1.016" layer="1"/>
+<wire x1="11.6586" y1="20.32" x2="14.1986" y2="20.32" width="1.016" layer="1"/>
+<wire x1="14.1986" y1="20.32" x2="14.1986" y2="23.9776" width="1.016" layer="1"/>
+<wire x1="14.1986" y1="23.9776" x2="14.224" y2="24.003" width="1.016" layer="1"/>
 </signal>
 <signal name="RED">
-<contactref element="R1" pad="2"/>
 <contactref element="U$1" pad="3"/>
 <contactref element="SL2" pad="3"/>
-<wire x1="21.5994" y1="26.0438" x2="19.4906" y2="26.0438" width="1.27" layer="1"/>
-<wire x1="19.4906" y1="26.0438" x2="15.4686" y2="22.0218" width="1.27" layer="1"/>
-<wire x1="15.4686" y1="22.0218" x2="15.4686" y2="20.9296" width="1.27" layer="1"/>
-<wire x1="15.4686" y1="20.9296" x2="15.4432" y2="20.9042" width="1.27" layer="1"/>
-<wire x1="15.4432" y1="20.9042" x2="15.4432" y2="16.7382" width="1.27" layer="1"/>
-<wire x1="15.4432" y1="16.7382" x2="16.764" y2="15.4174" width="1.27" layer="1"/>
+<wire x1="15.4432" y1="13.335" x2="15.4432" y2="18.6182" width="1.016" layer="1"/>
+<wire x1="15.4432" y1="18.6182" x2="21.5646" y2="24.7396" width="1.016" layer="1"/>
+<wire x1="21.5646" y1="24.7396" x2="21.5646" y2="26.009" width="1.016" layer="1"/>
+<wire x1="21.5646" y1="26.009" x2="21.5994" y2="26.0438" width="1.016" layer="1"/>
 </signal>
 <signal name="BLACK">
-<contactref element="R2" pad="2"/>
 <contactref element="U$2" pad="3"/>
 <contactref element="SL2" pad="1"/>
-<wire x1="2.5494" y1="26.1454" x2="2.5494" y2="23.5458" width="1.27" layer="1"/>
-<wire x1="2.5494" y1="23.5458" x2="10.3632" y2="23.5458" width="1.27" layer="1"/>
-<wire x1="10.3632" y1="23.5458" x2="10.3632" y2="20.9042" width="1.27" layer="1"/>
-<wire x1="10.3632" y1="20.9042" x2="10.3632" y2="16.8652" width="1.27" layer="1"/>
-<wire x1="10.3632" y1="16.8652" x2="8.6614" y2="15.1634" width="1.27" layer="1"/>
-</signal>
-<signal name="N$3">
-<contactref element="U$3" pad="1"/>
-<contactref element="R1" pad="1"/>
-<wire x1="14.0462" y1="12.4202" x2="16.8402" y2="12.5218" width="1.4224" layer="1"/>
-<wire x1="16.8402" y1="12.5218" x2="16.764" y2="12.5734" width="1.4224" layer="1"/>
-</signal>
-<signal name="N$4">
-<contactref element="U$4" pad="1"/>
-<contactref element="R2" pad="1"/>
-<wire x1="11.5824" y1="12.4202" x2="8.509" y2="12.344" width="1.4224" layer="1"/>
-<wire x1="8.509" y1="12.344" x2="8.6614" y2="12.3194" width="1.4224" layer="1"/>
+<wire x1="2.5494" y1="26.1454" x2="2.5494" y2="25.9494" width="1.016" layer="1"/>
+<wire x1="2.5494" y1="25.9494" x2="10.3886" y2="18.1102" width="1.016" layer="1"/>
+<wire x1="10.3886" y1="18.1102" x2="10.3886" y2="13.3604" width="1.016" layer="1"/>
+<wire x1="10.3886" y1="13.3604" x2="10.3632" y2="13.335" width="1.016" layer="1"/>
 </signal>
 </signals>
