File: circuits/In3Peltier/in3peltier.sch (EAGLE design)
At the start: 10 parts

Commit message: Electronics v2
Parts:
- removed R1, R2: 1M, 01_FAB_Hello:RESISTOR1206
- removed U$3, U$4: (no value), 01_FAB_Hello:LED1206
Connections:
- removed net N$3: R1.1, U$3.A
- removed net N$4: R2.1, U$4.A
- net BLACK: no longer R2.2
- net GNDH: no longer U$3.C, U$4.C
- net RED: no longer R1.2
Changed lines of the file:
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@@
 <part name="SL1" library="con-amp-quick" deviceset="MA03" device=""/>
 <part name="C1" library="01_SparkFun" deviceset="CAP_POL" device="PTH2"/>
-<part name="U$3" library="01_FAB_Hello" deviceset="LED" device="1206"/>
-<part name="U$4" library="01_FAB_Hello" deviceset="LED" device="1206"/>
-<part name="R1" library="01_FAB_Hello" deviceset="RESISTOR" device="1206" value="1M"/>
-<part name="R2" library="01_FAB_Hello" deviceset="RESISTOR" device="1206" value="1M"/>
 <part name="SL4" library="con-amp-quick" deviceset="MA03" device=""/>
 <part name="U$1" library="0001_alejandro" deviceset="RELAY-V23092" device="THROUGH_HOLE"/>
@@
 <instance part="SL1" gate="G$1" x="76.2" y="116.84"/>
 <instance part="C1" gate="G$1" x="63.5" y="96.52"/>
-<instance part="U$3" gate="G$1" x="-58.42" y="50.8"/>
-<instance part="U$4" gate="G$1" x="-43.18" y="50.8"/>
-<instance part="R1" gate="G$1" x="-58.42" y="66.04" rot="R90"/>
-<instance part="R2" gate="G$1" x="-43.18" y="66.04" rot="R90"/>
 <instance part="SL4" gate="G$1" x="30.48" y="96.52"/>
 <instance part="U$1" gate="G$1" x="-91.44" y="93.98"/>
@@
 <pinref part="U$2" gate="G$1" pin="1"/>
 </segment>
-<segment>
-<pinref part="U$3" gate="G$1" pin="C"/>
-<wire x1="-58.42" y1="48.26" x2="-58.42" y2="43.18" width="0.1524" layer="91"/>
-<pinref part="U$4" gate="G$1" pin="C"/>
-<wire x1="-58.42" y1="43.18" x2="-50.8" y2="43.18" width="0.1524" layer="91"/>
-<wire x1="-50.8" y1="43.18" x2="-43.18" y2="43.18" width="0.1524" layer="91"/>
-<wire x1="-43.18" y1="43.18" x2="-43.18" y2="48.26" width="0.1524" layer="91"/>
-<wire x1="-50.8" y1="43.18" x2="-50.8" y2="38.1" width="0.1524" layer="91"/>
-<junction x="-50.8" y="43.18"/>
-</segment>
 </net>
 <net name="RED" class="0">
@@
 <label x="-91.44" y="88.9" size="1.778" layer="95"/>
 <pinref part="U$1" gate="G$1" pin="3"/>
-</segment>
-<segment>
-<pinref part="R1" gate="G$1" pin="2"/>
-<wire x1="-58.42" y1="71.12" x2="-58.42" y2="76.2" width="0.1524" layer="91"/>
 </segment>
 </net>
@@
 <pinref part="U$2" gate="G$1" pin="3"/>
 </segment>
-<segment>
-<pinref part="R2" gate="G$1" pin="2"/>
-<wire x1="-43.18" y1="71.12" x2="-43.18" y2="76.2" width="0.1524" layer="91"/>
-</segment>
 </net>
-<net name="N$3" class="0">
-<segment>
-<pinref part="U$3" gate="G$1" pin="A"/>
-<pinref part="R1" gate="G$1" pin="1"/>
-<wire x1="-58.42" y1="55.88" x2="-58.42" y2="60.96" width="0.1524" layer="91"/>
-</segment>
-</net>
-<net name="N$4" class="0">
-<segment>
-<pinref part="U$4" gate="G$1" pin="A"/>
-<pinref part="R2" gate="G$1" pin="1"/>
-<wire x1="-43.18" y1="55.88" x2="-43.18" y2="60.96" width="0.1524" layer="91"/>
-</segment>
-</net>
