File: circuits/In3ControlPanel/in3controlpanel.sch (EAGLE design)
At the start: 27 parts, among them IC1 ATMEGA48/88/168-AU, SW1 EC12E_SW

Commit message: Electronics v2
Parts:
- removed C3: .1uf, ng:UNPOLARIZED_CAPACITOR1206
- removed C5: 10uf, ng:UNPOLARIZED_CAPACITOR1206
- removed IC1: ATMEGA48/88/168-AU, atmega8:ATMEGA48/88/168-AU
- removed LED: (no value), ng:LED1206
- removed SV3: (no value), con-lstb:MA06-1
- removed U$2: RESONATOREFOB, fab:RESONATOREFOB
- added R5: 0, ng:RESISTOR1206
- added SV1, SV2: (no value), con-lstb:MA05-2
- C1, C2: value (none) -> 0.01uf
- R2: value 499 -> 0
- R7: value 1k -> 0
- U$1: value AVRISPSMD -> (none); device 01_FAB_Hello:AVRISPSMD -> 01_adafruit:TRIMPOTTC33X
Connections:
- removed net 12V: SV3.4
- removed net ADC6: IC1.ADC6
- removed net MISO: IC1.PB4(MISO/PCINT4), U$1.MISO
- removed net MOSI: IC1.PB3(MOSI/OC2A/PCINT3), U$1.MOSI
- removed net N$1: IC1.PB7(XTAL2/TOSC2/PCINT7), U$2.1
- removed net N$23: LED.A, R2.2
- removed net N$9: IC1.PB6(XTAL1/TOSC1/PCINT6), U$2.3
- removed net PB0: IC1.PB0(ICP1/CLKO/PCINT0), SL1.3
- removed net PB1: IC1.PB1(OC1A/PCINT1), SL1.2
- removed net PB2: IC1.PB2(SS/OC1B/PCINT2), SL1.1
- removed net PC0: IC1.PC0(ADC0/PCINT8), R1.1
- removed net PC1: IC1.PC1(ADC1/PCINT9), R3.1
- removed net PC2: IC1.PC2(ADC2/PCINT10), R4.1
- removed net PD0: IC1.PD0(RXD/PCINT16)
- removed net PD1: IC1.PD1(TXD/PCINT17), SG1.1
- removed net PD5: IC1.PD5(T1/OC0B/PCINT21), SL1.11
- removed net PD6: IC1.PD6(AIN0/OC0A/PCINT22), SL1.9
- removed net PD7: IC1.PD7(AIN1/PCINT23), SL1.4
- removed net SCL: IC1.PC5(ADC5/SCL/PCINT13), SV3.3
- removed net SDA: IC1.PC4(ADC4/SDA/PCINT12), SV3.2
- removed net SWBUTTON: IC1.PD4(T0/XCK/PCINT20), R13.2, SW1G$2.1
- new net $1: SV2.5
- new net $2: SV2.6
- new net BTN: R13.2, R7.1, R7.2, SV2.4, SW1G$2.1
- new net BUZZ: SG1.1, SV1.2
- new net LCD4: R2.1, R2.2, SL1.4, SV2.8
- new net LCD5: SL1.3, SV2.10
- new net LCD6: SL1.2, SV2.9
- new net LCD7: SL1.1, SV2.7
- new net LCDE: SL1.9, SV1.3
- new net LCDRS: SL1.11, SV1.1
- new net RGBB: R3.1, SV1.6
- new net RGBG: R1.1, SV1.4
- net 5V: now also R5.1, R5.2, SV1.10, SV1.7, U$1.S; no longer C3.2, C5.2, IC1.AREF, IC1.AVCC, IC1.VCC@1, IC1.VCC@2, R7.2, R8.1, R8.2, SV3.5, U$1.VCC
- net GND: now also S1.P1, SV1.5; no longer C3.1, C5.1, IC1.AGND, IC1.GND@1, LED.C, SV3.6, U$1.GND, U$2.2
- net INT0: now also R8.1, R8.2, SV2.1; no longer IC1.PD2(INT0/PCINT18)
- net INT1: now also SV2.2; no longer IC1.PD3(INT1/OC2B/PCINT19)
- net N$6: now also U$1.E; no longer R7.1
- net RST: now also SV1.9, SV2.3; no longer IC1.PC6(/RESET/PCINT14), SV3.1, U$1.RST
- net SCK: now also R4.1, SV1.8; no longer IC1.PB5(SCK/PCINT5), R2.1, U$1.SCK
Other:
- moved on the sheet: R2, R7, R8

Commit message: New Electronics
Parts:
- removed R5, R7, R8: 0, ng:RESISTOR1206
- removed R6: 10k, ng:RESISTOR1206
- removed SL1: (no value), con-amp-quick:MA14
- removed SV1: (no value), con-lstb:MA05-2
- removed U$1: (no value), 01_adafruit:TRIMPOTTC33X
- added SL2: (no value), con-amp-quick:MA04
- LED1: device 01_fab:LEDRGBOLD -> eagle-ltspice:LED_E
- R1: value 1k -> 0R
- R3: value 470 -> 0
- SG1: value BUZZERNS -> F/CM12P; device 01_SparkFun:BUZZERNS -> buzzer:F/CM12P
Connections:
- removed net $1: SV2.5
- removed net $2: SV2.6
- removed net LCD4: R2.1, R2.2, SL1.4, SV2.8
- removed net LCD5: SL1.3, SV2.10
- removed net LCD6: SL1.2, SV2.9
- removed net LCD7: SL1.1, SV2.7
- removed net LCDE: SL1.9, SV1.3
- removed net LCDRS: SL1.11, SV1.1
- removed net N$2: LED1.CGREEN, R1.2
- removed net N$3: LED1.CBLUE, R3.2
- removed net N$4: LED1.CRED, R4.2
- removed net N$6: R6.2, SL1.12, U$1.E
- removed net RGBB: R3.1, SV1.6
- removed net RGBG: R1.1, SV1.4
- removed net SCK: R4.1, SV1.8
- new net LED: R4.1, SV2.10
- new net N$1: LED1.C, R4.2
- new net SCL: SL2.1, SV2.3
- new net SDA: SL2.2, SV2.5
- net 5V: now also LED1.A, SL2.3, SV2.7; no longer LED1.A2, R5.1, R5.2, SL1.13, SV1.10, SV1.7, U$1.S
- net BTN: no longer R7.1, R7.2
- net BUZZ: now also SV2.2; no longer SV1.2
- net GND: now also SL2.4, SV2.9; no longer R6.1, SL1.10, SL1.14, SV1.5
- net INT0: now also R1.1, R1.2, SV2.8; no longer R8.1, R8.2, SV2.1
- net INT1: now also R2.1, R2.2, SV2.6; no longer SV2.2
- net RST: now also R3.1, R3.2, SV2.1; no longer SV1.9, SV2.3
Other:
- moved on the sheet: C1, C2, R1, R10, R11, R12, R13, R14, R2, R3, R9, S1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
