File: circuits/In3Temperature/in3temperature.sch (EAGLE design)
At the start: 24 parts, among them IC1 ATMEGA48/88/168-AU, Q1 MOSFET-NCHANNELSMD, Q2 MOSFET-NCHANNELSMD, Q3 MOSFET-NCHANNELSMD, Q4 MOSFET-NCHANNELSMD, Q5 MOSFET-NCHANNELSMD

Commit message: Electronics v2
Parts:
- removed FAN1, FAN2: (no value), con-amp-quick:MA02
- removed SV1, SV3: (no value), con-lstb:MA06-1
- removed SV2, SV4: (no value), con-lstb:MA04-1
- added C6, C8: 10uf, ng:UNPOLARIZED_CAPACITOR1206
- added C7: .1uf, ng:UNPOLARIZED_CAPACITOR1206
- added IC2: REG1117, burr-brown:REG1117
- added R1, R3: 0, ng:RESISTOR1206
- added SL2, SL3: (no value), con-amp-quick:MA05
- added U$3, U$4: AVRISPSMD, 01_FAB_Hello:AVRISPSMD
Connections:
- net 12V: now also C6.2, C7.2, IC2.VIN, SL2.4, SL3.4, U$3.MISO; no longer FAN1.1, FAN2.1, SV1.4, SV3.4
- net 5V: now also C8.2, IC2.VOUT, R1.1, R1.2, R3.1, R3.2, U$3.RST, U$3.SCK, U$4.MOSI, U$4.SCK; no longer SV1.5, SV2.1, SV3.5, SV4.1
- net FAN1O: now also U$3.GND, U$3.MOSI; no longer FAN1.2
- net FAN2O: now also U$3.VCC; no longer FAN2.2
- net GND: now also C6.1, C7.1, C8.1, IC2.GND, SL2.5, SL3.5, U$4.MISO, U$4.VCC; no longer SV1.6, SV2.4, SV3.6, SV4.4
- net PD3: now also U$4.GND; no longer SV2.3
- net PD4: now also U$4.RST; no longer SV4.3
- net RST: now also SL2.1, SL3.1; no longer SV1.1, SV3.1
- net SCL: now also SL2.3, SL3.3; no longer SV1.3, SV3.3
- net SDA: now also SL2.2, SL3.2; no longer SV1.2, SV3.2

Commit message: New Electronics
Parts:
- removed C2: 1uf, ng:UNPOLARIZED_CAPACITOR1206
- removed C3, C7: .1uf, ng:UNPOLARIZED_CAPACITOR1206
- removed C4, C5, C6, C8: 10uf, ng:UNPOLARIZED_CAPACITOR1206
- removed IC1: ATMEGA48/88/168-AU, atmega8:ATMEGA48/88/168-AU
- removed IC2: REG1117, burr-brown:REG1117
- removed LED: (no value), ng:LED1206
- removed R1, R3, R7: 0, ng:RESISTOR1206
- removed R2: 499, ng:RESISTOR1206
- removed SL1: (no value), con-amp-quick:MA03
- removed U$4: AVRISPSMD, 01_FAB_Hello:AVRISPSMD
- added D1, D2, D3: (no value), fab:ZENER_DIODESOD123
- added J1: (no value), con-jack:JACK-PLUG1
- C1: value 1uf -> (none); device ng:UNPOLARIZED_CAPACITOR1206 -> resistor:CPOL-USE2.5-5
- SL2: device con-amp-quick:MA05 -> con-amp-quick:MA07
- SL3: device con-amp-quick:MA05 -> con-amp-quick:MA03
- U$1: value AVRISPSMD -> RELAY-V23092THROUGH_HOLE; device 01_FAB_Hello:AVRISPSMD -> 0001_alejandro:RELAY-V23092THROUGH_HOLE
- U$2: value RESONATOREFOB -> RELAY-V23092THROUGH_HOLE; device fab:RESONATOREFOB -> 0001_alejandro:RELAY-V23092THROUGH_HOLE
Connections:
- removed net 5V: C2.2, C3.2, C5.2, C8.2, IC1.AREF, IC1.AVCC, IC1.VCC@1, IC1.VCC@2, IC2.VOUT, R1.1, R1.2, R3.1, R3.2, U$1.VCC, U$3.RST, U$3.SCK, U$4.MOSI, U$4.SCK
- removed net FAN1: IC1.PD6(AIN0/OC0A/PCINT22), Q1.G
- removed net FAN2: IC1.PD5(T1/OC0B/PCINT21), Q2.G
- removed net MISO: IC1.PB4(MISO/PCINT4), U$1.MISO
- removed net MOSI: IC1.PB3(MOSI/OC2A/PCINT3), U$1.MOSI
- removed net N$1: IC1.PB7(XTAL2/TOSC2/PCINT7), U$2.1
- removed net N$23: LED.A, R2.2
- removed net N$9: IC1.PB6(XTAL1/TOSC1/PCINT6), U$2.3
- removed net PD0: IC1.PD0(RXD/PCINT16), Q5.G
- removed net PD3: IC1.PD3(INT1/OC2B/PCINT19), U$4.GND
- removed net PD4: IC1.PD4(T0/XCK/PCINT20), U$4.RST
- removed net RST: IC1.PC6(/RESET/PCINT14), R7.1, R7.2, SL2.1, SL3.1, U$1.RST
- removed net SCK: IC1.PB5(SCK/PCINT5), R2.1, U$1.SCK
- removed net SCL: IC1.PC5(ADC5/SCL/PCINT13), SL2.3, SL3.3
- removed net SDA: IC1.PC4(ADC4/SDA/PCINT12), SL2.2, SL3.2
- new net BLACK: SL3.1, U$2.3
- new net FAN12: Q2.G, SL2.5
- new net FAN5: Q1.G, SL2.4
- new net PUMP: Q5.G, SL2.1
- new net RED: SL3.3, U$1.3
- net 12V: now also C1.+, D1.CATHODE, D2.CATHODE, D3.CATHODE, J1.3, SL2.7, U$1.2, U$1.4, U$2.2, U$2.4, U$3.RST, U$3.SCK; no longer C1.2, C4.2, C6.2, C7.2, IC2.VIN, SL1.2, SL2.4, SL3.4
- net FAN1O: now also D2.ANODE
- net FAN2O: now also D1.ANODE
- net GND: now also C1.-, J1.1, J1.2, SL2.6, U$1.1, U$2.1; no longer C1.1, C2.1, C3.1, C4.1, C5.1, C6.1, C7.1, C8.1, IC1.AGND, IC1.GND@1, IC2.GND, LED.C, SL2.5, SL3.5, U$1.GND, U$2.2, U$4.MISO, U$4.VCC
- net N$3: now also D3.ANODE
- net RELAY1: now also SL2.3; no longer IC1.PD1(TXD/PCINT17)
- net RELAY1O: now also U$1.5; no longer SL1.3
- net RELAY2: now also SL2.2; no longer IC1.PD2(INT0/PCINT18)
- net RELAY2O: now also U$2.5; no longer SL1.1
Other:
- moved on the sheet: Q3, Q4
