File: circuits/In3Brain/in3brain.sch (EAGLE design)
At the start: 21 parts, among them IC1 ATMEGA48/88/168-AU, IC2 REG1117

Commit message: Electronics v2
Parts:
- removed LED: (no value), ng:LED1206
- removed R9: 0, ng:RESISTOR1206
- removed S1: (no value), ng:6MM_SWITCH6MM_SWITCH
- removed SV2, SV3: (no value), con-lstb:MA06-1
- added J1: JACK.65MM, 01_fab:JACK.65MM
- added SV5, SV6: (no value), con-lstb:MA05-2
- R1: value 10k -> 0
- R2: value 499 -> 0
- SL1: device con-amp-quick:MA02 -> con-amp-quick:MA05
Connections:
- removed net EN: SV2.1
- removed net N$23: LED.A, R2.2
- new net $1: SV5.5
- new net $2: SV5.6
- new net BTN: IC1.PD4(T0/XCK/PCINT20), SV5.4
- new net BUZZ: IC1.PB0(ICP1/CLKO/PCINT0), SV6.2
- new net INT0: IC1.PD2(INT0/PCINT18), SV5.1
- new net INT1: IC1.PD3(INT1/OC2B/PCINT19), SV5.2
- new net LCD4: IC1.PC0(ADC0/PCINT8), SV5.8
- new net LCD5: IC1.PC1(ADC1/PCINT9), SV5.10
- new net LCD6: IC1.PC2(ADC2/PCINT10), SV5.9
- new net LCD7: IC1.PC3(ADC3/PCINT11), SV5.7
- new net LCDE: IC1.PD6(AIN0/OC0A/PCINT22), SV6.3
- new net LCDRS: IC1.PD7(AIN1/PCINT23), SV6.1
- new net RGBB: IC1.PB2(SS/OC1B/PCINT2), SV6.6
- new net RGBG: IC1.PB1(OC1A/PCINT1), SV6.4
- net 12V: now also J1.PIN, SL1.4; no longer SL1.1, SV3.4
- net 5V: now also R2.1, R2.2, SV6.10, SV6.7; no longer R1.2, R9.1, R9.2, SV2.2, SV3.5
- net GND: now also J1.CONTACT, J1.SHUNT, R1.1, R1.2, SL1.5, SV6.5; no longer LED.C, S1.P, S1.P1, SL1.2, SV2.3, SV3.6
- net RST: now also SL1.1, SV5.3, SV6.9; no longer R1.1, S1.S, S1.S1, SV3.1
- net RX: no longer SV2.6
- net SCK: now also SV6.8; no longer R2.1
- net SCL: now also SL1.3; no longer SV3.3
- net SDA: now also SL1.2; no longer SV3.2
- net STATE: now also IC1.PD5(T1/OC0B/PCINT21); no longer IC1.PD4(T0/XCK/PCINT20), SV2.4
- net TX: no longer SV2.5
Other:
- moved on the sheet: R1, R2

Commit message: New Electronics
Parts:
- removed J1: JACK.65MM, 01_fab:JACK.65MM
- removed R7, R8: 0, ng:RESISTOR1206
- removed SV5: (no value), con-lstb:MA05-2
- added J2: (no value), con-jack:JACK-PLUG1
- added R5: 0, ng:RESISTOR1206
- added SL2, SL3: (no value), con-amp-quick:MA03
- added SL5: (no value), con-amp-quick:MA07
Connections:
- removed net $1: SV5.5
- removed net $2: SV5.6
- removed net LCD4: IC1.PC0(ADC0/PCINT8), SV5.8
- removed net LCD5: IC1.PC1(ADC1/PCINT9), SV5.10
- removed net LCD6: IC1.PC2(ADC2/PCINT10), SV5.9
- removed net LCD7: IC1.PC3(ADC3/PCINT11), SV5.7
- removed net LCDE: IC1.PD6(AIN0/OC0A/PCINT22), SV6.3
- removed net LCDRS: IC1.PD7(AIN1/PCINT23), SV6.1
- removed net RGBB: IC1.PB2(SS/OC1B/PCINT2), SV6.6
- removed net RGBG: IC1.PB1(OC1A/PCINT1), SV6.4
- removed net RX: IC1.PD0(RXD/PCINT16)
- removed net STATE: IC1.PD5(T1/OC0B/PCINT21)
- removed net TX: IC1.PD1(TXD/PCINT17)
- new net FAN12: IC1.PD5(T1/OC0B/PCINT21), SL5.5
- new net FAN5: IC1.PD6(AIN0/OC0A/PCINT22), SL5.4
- new net LED: IC1.PD4(T0/XCK/PCINT20), SV6.10
- new net PUMP: IC1.PB1(OC1A/PCINT1), SL5.1
- new net RELAY1: IC1.PD7(AIN1/PCINT23), SL5.3
- new net RELAY2: IC1.PB0(ICP1/CLKO/PCINT0), SL5.2
- new net TEMP1: IC1.PC0(ADC0/PCINT8), SL2.1
- new net TEMP2: IC1.PC1(ADC1/PCINT9), SL3.1
- net 12V: now also J2.3, SL1.5, SL5.7; no longer J1.PIN, SL1.4
- net 5V: now also SL2.3, SL3.3; no longer R8.1, R8.2, SV6.10
- net BTN: now also IC1.PD1(TXD/PCINT17), SV6.4; no longer IC1.PD4(T0/XCK/PCINT20), SV5.4
- net BUZZ: now also IC1.PD0(RXD/PCINT16); no longer IC1.PB0(ICP1/CLKO/PCINT0)
- net GND: now also IC1.GND@2, J2.1, J2.2, R5.1, R5.2, SL1.2, SL2.2, SL3.2, SL5.6, SV6.9; no longer J1.CONTACT, J1.SHUNT, R1.1, R1.2, SL1.5, SV6.5
- net INT0: now also IC1.PD3(INT1/OC2B/PCINT19), SV6.8; no longer IC1.PD2(INT0/PCINT18), SV5.1
- net INT1: now also IC1.PD2(INT0/PCINT18), SV6.6; no longer IC1.PD3(INT1/OC2B/PCINT19), SV5.2
- net MISO: now also R1.1, R1.2
- net RST: now also IC1.ADC6, SV6.1; no longer R7.1, R7.2, SV5.3, SV6.9
- net SCK: no longer SV6.8
- net SCL: now also SV6.3
- net SDA: now also SL1.4, SV6.5; no longer SL1.2
Other:
- note added: "Connection header"
- moved on the sheet: R1, R2, R3, R4, SL1

Commit message: new electronics: less components, less bards, space optimization and some software error fixes
Parts:
- removed C3: .1uf, ng:UNPOLARIZED_CAPACITOR1206
- removed C5, C6: 10uf, ng:UNPOLARIZED_CAPACITOR1206
- removed IC1: ATMEGA48/88/168-AU, atmega8:ATMEGA48/88/168-AU
- removed IC2: REG1117, burr-brown:REG1117
- removed J2: (no value), con-jack:JACK-PLUG1
- removed R5: 0, ng:RESISTOR1206
- removed SL5: (no value), con-amp-quick:MA07
- removed SV6: (no value), con-lstb:MA05-2
- removed U$1: AVRISPSMD, 01_FAB_Hello:AVRISPSMD
- removed U$2: RESONATOREFOB, fab:RESONATOREFOB
- added C10, C9: .1uf, ng:UNPOLARIZED_CAPACITOR1206
- added C11, C12: 10uf, ng:UNPOLARIZED_CAPACITOR1206
- added C8: 1uf, ng:UNPOLARIZED_CAPACITOR1206
- added IC3: ATMEGA48/88/168-AU, atmega8:ATMEGA48/88/168-AU
- added IC4: REG1117, burr-brown:REG1117
- added J1: (no value), con-jack:JACK-PLUG1
- added LED1, LED2: (no value), eagle-ltspice:LED_E
- added R10, R11, R12, R13, R14, R16, R17, R9: 10k, ng:RESISTOR1206
- added S1: (no value), 01_FAB_Hello:6MM_SWITCH6MM_SWITCH
- added SG1: F/CM12P, buzzer:F/CM12P
- added SL4: (no value), con-amp-quick:MA08
- added SL7, SL8: (no value), con-amp-quick:MA03
- added SW1: EC12E_SW, switch-alps:EC12E_SW
- added U$3: RESONATOREFOB, fab:RESONATOREFOB
- added U$4: AVRISPSMD, 01_FAB_Hello:AVRISPSMD
- C1: value .1uf -> 0.01uf; device ng:UNPOLARIZED_CAPACITOR1206 -> 01_FAB_Hello:UNPOLARIZED_CAPACITOR1206
- C2: value 1uf -> 0.01uf; device ng:UNPOLARIZED_CAPACITOR1206 -> 01_FAB_Hello:UNPOLARIZED_CAPACITOR1206
- R2: value 0 -> 499
- R3: value 10k -> 0
- R4: value 10k -> 499
- SL1: device con-amp-quick:MA05 -> con-amp-quick:MA06
- SL2: device con-amp-quick:MA03 -> con-amp-quick:MA04
- SL3: device con-amp-quick:MA03 -> con-amp-quick:MA05
Connections:
- removed net AREF: IC1.AREF
- removed net N$9: IC1.PB6(XTAL1/TOSC1/PCINT6), U$2.3
- new net ADC2: IC3.PC2(ADC2/PCINT10), SL4.1
- new net CTS: SL1.2
- new net N$2: LED2.C, R2.2
- new net N$3: IC3.PB7(XTAL2/TOSC2/PCINT7), U$3.1
- new net N$4: IC3.PB6(XTAL1/TOSC1/PCINT6), U$3.3
- new net N$5: R11.2, R9.1, SW1G$1.B
- new net N$8: R10.2, R12.2, SW1G$1.A
- new net RX: IC3.PD0(RXD/PCINT16), SL1.4
- new net TX: IC3.PD1(TXD/PCINT17), SL1.5
- net 12V: now also C10.2, C11.2, IC4.VIN, J1.3, SL3.1, SL4.8; no longer C1.2, C5.2, IC2.VIN, J2.3, SL1.5, SL5.7
- net 5V: now also C12.2, C8.2, C9.2, IC3.AREF, IC3.AVCC, IC3.VCC@1, IC3.VCC@2, IC4.VOUT, LED1.A, LED2.A, R11.1, R12.1, R13.1, R14.2, R16.1, R17.1, R3.2, SL1.3, SL7.3, SL8.3, U$4.VCC; no longer C2.2, C3.2, C6.2, IC1.AVCC, IC1.VCC@1, IC1.VCC@2, IC2.VOUT, R2.1, R2.2, R4.1, SL3.3, SV6.7, U$1.VCC
- net BTN: now also IC3.ADC7, R13.2, SW1G$2.1; no longer IC1.PD1(TXD/PCINT17), SV6.4
- net BUZZ: now also IC3.ADC6, SG1.1; no longer IC1.PD0(RXD/PCINT16), SV6.2
- net FAN12: now also IC3.PD5(T1/OC0B/PCINT21), SL4.6; no longer IC1.PD5(T1/OC0B/PCINT21), SL5.5
- net FAN5: now also IC3.PD6(AIN0/OC0A/PCINT22), SL4.5; no longer IC1.PD6(AIN0/OC0A/PCINT22), SL5.4
- net GND: now also C10.1, C11.1, C12.1, C8.1, C9.1, IC3.AGND, IC3.GND@1, IC3.GND@2, IC4.GND, J1.1, J1.2, R1.1, R1.2, S1.P, S1.P1, SG1.2, SL1.1, SL2.4, SL3.3, SL4.7, SL7.2, SL8.2, SW1G$1.C, SW1G$2.2, U$3.2, U$4.GND; no longer C3.1, C5.1, C6.1, IC1.AGND, IC1.GND@1, IC1.GND@2, IC2.GND, J2.1, J2.2, R5.1, R5.2, SL1.2, SL2.2, SL3.2, SL5.6, SV6.9, U$1.GND, U$2.2
- net INT0: now also C1.2, IC3.PD3(INT1/OC2B/PCINT19), R10.1; no longer IC1.PD3(INT1/OC2B/PCINT19), SV6.8
- net INT1: now also C2.2, IC3.PD2(INT0/PCINT18), R9.2; no longer IC1.PD2(INT0/PCINT18), SV6.6
- net LED: now also IC3.PD4(T0/XCK/PCINT20), R4.1; no longer IC1.PD4(T0/XCK/PCINT20), SV6.10
- net MISO: now also IC3.PB4(MISO/PCINT4), U$4.MISO; no longer IC1.PB4(MISO/PCINT4), R1.1, R1.2, U$1.MISO
- net MOSI: now also IC3.PB3(MOSI/OC2A/PCINT3), U$4.MOSI; no longer IC1.PB3(MOSI/OC2A/PCINT3), U$1.MOSI
- net N$1: now also LED1.C, R4.2; no longer IC1.PB7(XTAL2/TOSC2/PCINT7), U$2.1
- net PUMP: now also IC3.PB1(OC1A/PCINT1), SL4.2; no longer IC1.PB1(OC1A/PCINT1), SL5.1
- net RELAY1: now also IC3.PD7(AIN1/PCINT23), SL4.4; no longer IC1.PD7(AIN1/PCINT23), SL5.3
- net RELAY2: now also IC3.PB0(ICP1/CLKO/PCINT0), SL4.3; no longer IC1.PB0(ICP1/CLKO/PCINT0), SL5.2
- net RST: now also IC3.PC6(/RESET/PCINT14), R14.1, S1.S, S1.S1, SL1.6, SL3.2, U$4.RST; no longer IC1.ADC6, IC1.PC6(/RESET/PCINT14), SL1.1, SV6.1, U$1.RST
- net SCK: now also IC3.PB5(SCK/PCINT5), R2.1, U$4.SCK; no longer IC1.PB5(SCK/PCINT5), U$1.SCK
- net SCL: now also IC3.PC5(ADC5/SCL/PCINT13), R16.2, SL2.1, SL3.4; no longer IC1.PC5(ADC5/SCL/PCINT13), R3.2, SL1.3, SV6.3
- net SDA: now also IC3.PC4(ADC4/SDA/PCINT12), R17.2, SL2.2, SL3.5; no longer IC1.PC4(ADC4/SDA/PCINT12), R4.2, SL1.4, SV6.5
- net TEMP1: now also IC3.PC0(ADC0/PCINT8), SL7.1; no longer IC1.PC0(ADC0/PCINT8), SL2.1
- net TEMP2: now also IC3.PC1(ADC1/PCINT9), SL8.1; no longer IC1.PC1(ADC1/PCINT9), SL3.1
Other:
- moved on the sheet: C1, C2, R1, R2, R3, R4
